File: the Ducker Doodle/the Ducker Doodle.kicad_pcb (KiCad board)
At the start: 2 copper layers, 210 parts, among them J1 USB_C, U2 USBLC6-2SC6, U3 XC6206

Commit message: feat: updated pcb
Parts:
- added U1: ATMEGA32U4-MU, Microchip Tech ATMEGA32U4-MU:44PW_ATM, B.Cu at (190.4, 145.5)
- C1, C2, C3, C4, F1, FB1, FB2, J1, R1, R2, R3, R_BUTT1, U2, U3: moved to B.Cu
- moved C3 149.1 mm to (193.5, 151.0), turned to 180 degrees
- moved J1 147.2 mm to (200.7, 133.1)
- moved F1 144.8 mm to (205.0, 140.0), turned to -90 degrees
- moved C2 141.2 mm to (188.0, 151.0)
- moved R1 139.9 mm to (207.0, 134.5), turned to -90 degrees
- moved C4 138.9 mm to (194.0, 140.0), turned to 180 degrees
- moved U3 138.5 mm to (204.0, 143.9), turned to 90 degrees
- moved U2 137.3 mm to (199.9, 141.1), turned to 90 degrees
- moved R_BUTT1 134.9 mm to (176.1, 143.8), turned to 90 degrees
- moved FB2 133.8 mm to (183.0, 147.0), turned to 90 degrees
- moved C1 133.4 mm to (187.5, 140.0), turned to 180 degrees
- moved FB1 131.9 mm to (183.0, 142.2), turned to -90 degrees
- moved R3 131.3 mm to (175.0, 149.0), turned to 180 degrees
- moved R2 130.3 mm to (194.0, 134.5), turned to -90 degrees
- moved D13 121.0 mm to (490.8, 142.9)
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Routing:
- net COL_20: track 111.7 -> 64.1 mm
- net Net-(D66-A): track 8.27 -> 0.00 mm
- net Net-(D22-A): track 8.27 -> 0.00 mm
- net Net-(D21-A): track 8.27 -> 0.00 mm
- net COL_16: track 119.6 -> 121.6 mm
- net ROW_6: track 315.9 -> 317.8 mm
Other:
- board outline added: 399 x 132 mm
