File: the Ducker Doodle/the Ducker Doodle.kicad_sch (KiCad schematic)
At the start: 0 parts

Commit message: feat: added switch matrix and usb stuff
Parts:
- added C1, C2: 1uF, ScottoKeebs_Components:Capacitor_0402, symbol Device:C_Small
- added D10, D100, D101, D102, D103, D104, D107, D108, D11, D111, D112, D113, D114, D115, D116, D117, D118, D119, D12, D120, D121, D122, D123, D125, D131, D132, D133, D134, D136, D139, D14, D143, D144, D146, D147, D15, D16, D17, D18, D19, D20, D21, D22, D23, D24, D25, D43, D44, D45, D46, D48, D49, D50, D51, D52, D53, D54, D55, D56, D57, D58, D59, D60, D61, D63, D64, D65, D66, D69, D7, D70, D72, D73, D74, D75, D76, D77, D78, D79, D80, D81, D82, D83, D84, D85, D86, D87, D88, D9, D90, D91, D93, D94, D95, D96, D97, D98, D99: Diode, symbol ScottoKeebs:Placeholder_Diode
- added F1: 500mA, ScottoKeebs_Components:Fuse_0603, symbol Device:Fuse_Small
- added J1: USB_C, ScottoKeebs_Components:USB_C_HRO_TYPE-C-31-M-12, symbol Connector:USB_C_Receptacle_USB2.0_14P
- added R1, R2: 5.1k, Resistor_SMD:R_0402_1005Metric, symbol Device:R_Small
- added R3: 10k, Resistor_SMD:R_0402_1005Metric, symbol Device:R_Small
- added S10, S100, S101, S102, S103, S104, S107, S108, S11, S111, S112, S113, S114, S115, S116, S117, S118, S119, S12, S120, S121, S122, S123, S125, S131, S132, S133, S134, S136, S139, S14, S143, S144, S146, S147, S15, S16, S17, S18, S19, S20, S21, S22, S23, S24, S25, S43, S44, S45, S46, S48, S49, S50, S51, S52, S53, S54, S55, S56, S57, S58, S59, S60, S61, S63, S64, S65, S66, S69, S7, S70, S72, S73, S74, S75, S76, S77, S78, S79, S80, S81, S82, S83, S84, S85, S86, S87, S88, S9, S90, S91, S93, S94, S95, S96, S97, S98, S99: Keyswitch, symbol ScottoKeebs:Placeholder_Keyswitch
- added SW1: SW_Push, ScottoKeebs_Components:Button_TL3342, symbol Switch:SW_Push
- added U1: ATMEGA32U4-MU, 44PW_ATM, symbol Microchip Tech ATMEGA32U4-MU:ATMEGA32U4-MU
- added U2: USBLC6-2SC6, ScottoKeebs_Components:ESD_SOT-23-6, symbol Power_Protection:USBLC6-2SC6
- added U3: XC6206, ScottoKeebs_Components:Voltage_SOT-23, symbol Regulator_Linear:XC6206PxxxMR
Connections:
- new net: D108.2 (A), S108.2
- new net: D88.2 (A), S88.2
- new net: D50.2 (A), S50.2
- new net: D101.2 (A), S101.2
- new net: D70.2 (A), S70.2
- new net: D45.2 (A), S45.2
- new net: D104.2 (A), S104.2
- new net: D85.2 (A), S85.2
- new net: D25.2 (A), S25.2
- new net: D107.2 (A), S107.2
- new net: D79.2 (A), S79.2
- new net: D119.2 (A), S119.2
- new net: D69.2 (A), S69.2
- new net: D76.2 (A), S76.2
- new net: D78.2 (A), S78.2
- new net: J1.A5 (CC1), R1.1
- new net: D19.2 (A), S19.2
- new net: D82.2 (A), S82.2
- new net: D125.2 (A), S125.2
- new net: D9.2 (A), S9.2
- new net: D65.2 (A), S65.2
- new net: D57.2 (A), S57.2
- new net: D98.2 (A), S98.2
- new net: D66.2 (A), S66.2
- new net: D115.2 (A), S115.2
- new net: D133.2 (A), S133.2
- new net: D48.2 (A), S48.2
- new net: D53.2 (A), S53.2
- new net: D120.2 (A), S120.2
- new net: D103.2 (A), S103.2
- new net: D146.2 (A), S146.2
- new net: D52.2 (A), S52.2
- new net: D7.2 (A), S7.2
- new net: D22.2 (A), S22.2
- new net: D49.2 (A), S49.2
- new net: D73.2 (A), S73.2
- new net: D114.2 (A), S114.2
- new net: D23.2 (A), S23.2
- new net: D96.2 (A), S96.2
- new net: D74.2 (A), S74.2
- new net: D134.2 (A), S134.2
- new net: D116.2 (A), S116.2
- new net: D15.2 (A), S15.2
- new net: D118.2 (A), S118.2
- new net: D72.2 (A), S72.2
- new net: D84.2 (A), S84.2
- new net: D75.2 (A), S75.2
- new net: D131.2 (A), S131.2
- new net: D16.2 (A), S16.2
- new net: D64.2 (A), S64.2
- new net: D100.2 (A), S100.2
- new net: D14.2 (A), S14.2
- new net: D20.2 (A), S20.2
- new net: D11.2 (A), S11.2
- new net: D80.2 (A), S80.2
- new net: D12.2 (A), S12.2
- new net: D97.2 (A), S97.2
- new net: D144.2 (A), S144.2
- new net: J1.B5 (CC2), R2.1
- new net: D59.2 (A), S59.2
- new net: D10.2 (A), S10.2
- new net: D113.2 (A), S113.2
- new net: D61.2 (A), S61.2
- new net: D77.2 (A), S77.2
- new net: D63.2 (A), S63.2
- new net: D17.2 (A), S17.2
- new net: D24.2 (A), S24.2
- new net: D147.2 (A), S147.2
- new net: D54.2 (A), S54.2
- new net: D93.2 (A), S93.2
- new net: D46.2 (A), S46.2
- new net: D44.2 (A), S44.2
- new net: D83.2 (A), S83.2
- new net: D99.2 (A), S99.2
- new net: D117.2 (A), S117.2
- new net: D132.2 (A), S132.2
- new net: D86.2 (A), S86.2
- new net: D122.2 (A), S122.2
- new net: D81.2 (A), S81.2
- new net: D56.2 (A), S56.2
- new net: D18.2 (A), S18.2
- new net: D51.2 (A), S51.2
- new net: D112.2 (A), S112.2
- new net: D102.2 (A), S102.2
- new net: D58.2 (A), S58.2
- new net: D143.2 (A), S143.2
- new net: D139.2 (A), S139.2
- new net: D43.2 (A), S43.2
- new net: D87.2 (A), S87.2
- new net: D55.2 (A), S55.2
- new net: D60.2 (A), S60.2
- new net: D94.2 (A), S94.2
- new net: D21.2 (A), S21.2
- new net: D123.2 (A), S123.2
- new net: D111.2 (A), S111.2
- new net: D90.2 (A), S90.2
- new net: D136.2 (A), S136.2
- new net: D91.2 (A), S91.2
- new net: D121.2 (A), S121.2
- new net: D95.2 (A), S95.2
- new net +3.3V: C2.1, SW1.1, U3.2 (VO)
- new net +5V: C1.1, F1.2, U3.3 (VI)
- new net BOOT0: R3.2, SW1.2, U1.13 (*RESET)
- new net COL_0: S22.1, S43.1, S64.1, S85.1, U1.12 (PB7)
- new net COL_1: S107.1, S23.1, S44.1, S65.1, S86.1
- new net COL_10: S11.1, S116.1, S53.1, S74.1, S95.1
- new net COL_11: S117.1, S12.1, S54.1, S75.1, S96.1
- new net COL_12: S118.1, S139.1, S55.1, S76.1, S97.1
- new net COL_13: S119.1, S14.1, S56.1, S77.1, S98.1
- new net COL_14: S120.1, S15.1, S57.1, S78.1, S99.1
- new net COL_15: S100.1, S121.1, S16.1, S58.1, S79.1
- new net COL_16: S101.1, S122.1, S143.1, S17.1, S59.1, S80.1
- new net COL_17: S102.1, S123.1, S144.1, S18.1, S60.1, S81.1
- new net COL_18: S103.1, S19.1, S61.1, S82.1
- new net COL_19: S104.1, S125.1, S146.1, S20.1, S83.1
- new net COL_2: S108.1, S24.1, S45.1, S66.1, S87.1
- new net COL_20: S147.1, S21.1, S63.1, S84.1
- new net COL_3: S25.1, S46.1, S88.1
- new net COL_4: S131.1
- new net COL_5: S111.1, S132.1, S48.1, S69.1, S90.1
- new net COL_6: S112.1, S133.1, S49.1, S7.1, S70.1, S91.1
- new net COL_7: S113.1, S134.1, S50.1
- new net COL_8: S114.1, S51.1, S72.1, S9.1, S93.1
- new net COL_9: S10.1, S115.1, S136.1, S52.1, S73.1, S94.1
- new net GND: C1.2, C2.2, J1.A1 (GND), J1.A12 (GND), J1.B1 (GND), J1.B12 (GND), J1.S1 (SHIELD), R1.2, R2.2, R3.1, U2.2 (GND), U3.1 (GND)
- new net MCU_D+: U1.4 (D+), U2.1 (I/O1)
- new net MCU_D-: U1.3 (D-), U2.3 (I/O2)
- new net ROW_0: D10.1 (K), D11.1 (K), D12.1 (K), D14.1 (K), D15.1 (K), D16.1 (K), D17.1 (K), D18.1 (K), D19.1 (K), D20.1 (K), D21.1 (K), D7.1 (K), D9.1 (K), U1.10 (PB2), U1.11 (PB3), U1.28 (PB4), U1.29 (PB5), U1.30 (PB6), U1.8 (PB0), U1.9 (PB1)
- new net ROW_1: D22.1 (K), D23.1 (K), D24.1 (K), D25.1 (K)
- new net ROW_2: D43.1 (K), D44.1 (K), D45.1 (K), D46.1 (K), D48.1 (K), D49.1 (K), D50.1 (K), D51.1 (K), D52.1 (K), D53.1 (K), D54.1 (K), D55.1 (K), D56.1 (K), D57.1 (K), D58.1 (K), D59.1 (K), D60.1 (K), D61.1 (K), D63.1 (K)
- new net ROW_3: D64.1 (K), D65.1 (K), D66.1 (K), D69.1 (K), D70.1 (K), D72.1 (K), D73.1 (K), D74.1 (K), D75.1 (K), D76.1 (K), D77.1 (K), D78.1 (K), D79.1 (K), D80.1 (K), D81.1 (K), D82.1 (K), D83.1 (K), D84.1 (K)
- new net ROW_4: D100.1 (K), D101.1 (K), D102.1 (K), D103.1 (K), D104.1 (K), D85.1 (K), D86.1 (K), D87.1 (K), D88.1 (K), D90.1 (K), D91.1 (K), D93.1 (K), D94.1 (K), D95.1 (K), D96.1 (K), D97.1 (K), D98.1 (K), D99.1 (K)
- new net ROW_5: D107.1 (K), D108.1 (K), D111.1 (K), D112.1 (K), D113.1 (K), D114.1 (K), D115.1 (K), D116.1 (K), D117.1 (K), D118.1 (K), D119.1 (K), D120.1 (K), D121.1 (K), D122.1 (K), D123.1 (K), D125.1 (K)
- new net ROW_6: D131.1 (K), D132.1 (K), D133.1 (K), D134.1 (K), D136.1 (K), D139.1 (K), D143.1 (K), D144.1 (K), D146.1 (K), D147.1 (K)
- new net USB_D+: J1.A6 (D+), J1.B6 (D+), U2.6 (I/O1)
- new net USB_D-: J1.A7 (D-), J1.B7 (D-), U2.4 (I/O2)
- new net VBUS: F1.1, J1.A4 (VBUS), J1.A9 (VBUS), J1.B4 (VBUS), J1.B9 (VBUS), U2.5 (VBUS)
Other:
- note added: "Bootloader Button"
- note added: "ESD Protection"
- note added: "USB-C connector"
- note added: "Voltage Step Down"

Commit message: feat: updated pcb
Parts:
- added C1, C2: 1uF, ScottoKeebs_Components:Capacitor_0402, symbol Device:C_Small
- added FB1, FB2: MMZ1608A252BTA00, Resistor_SMD:R_0603_1608Metric, symbol Device:FerriteBead
- D1: renamed from D7; footprint (none) -> ScottoKeebs_Components:Diode_SOD-123
- D10: renamed from D18; footprint (none) -> ScottoKeebs_Components:Diode_SOD-123
- D11: renamed from D19; footprint (none) -> ScottoKeebs_Components:Diode_SOD-123
- D12: renamed from D20; footprint (none) -> ScottoKeebs_Components:Diode_SOD-123
- D13: renamed from D21; footprint (none) -> ScottoKeebs_Components:Diode_SOD-123
- D14: renamed from D22; footprint (none) -> ScottoKeebs_Components:Diode_SOD-123
- D15: renamed from D23; footprint (none) -> ScottoKeebs_Components:Diode_SOD-123
- D16: renamed from D24; footprint (none) -> ScottoKeebs_Components:Diode_SOD-123
- D17: renamed from D25; footprint (none) -> ScottoKeebs_Components:Diode_SOD-123
- D18: renamed from D43; footprint (none) -> ScottoKeebs_Components:Diode_SOD-123
- D19: renamed from D44; footprint (none) -> ScottoKeebs_Components:Diode_SOD-123
- D2: renamed from D9; footprint (none) -> ScottoKeebs_Components:Diode_SOD-123
- D20: renamed from D45; footprint (none) -> ScottoKeebs_Components:Diode_SOD-123
- D21: renamed from D46; footprint (none) -> ScottoKeebs_Components:Diode_SOD-123
- D22: renamed from D48; footprint (none) -> ScottoKeebs_Components:Diode_SOD-123
- D23: renamed from D49; footprint (none) -> ScottoKeebs_Components:Diode_SOD-123
- D24: renamed from D50; footprint (none) -> ScottoKeebs_Components:Diode_SOD-123
- D25: renamed from D51; footprint (none) -> ScottoKeebs_Components:Diode_SOD-123
- D26: renamed from D52; footprint (none) -> ScottoKeebs_Components:Diode_SOD-123
- D27: renamed from D53; footprint (none) -> ScottoKeebs_Components:Diode_SOD-123
- D28: renamed from D54; footprint (none) -> ScottoKeebs_Components:Diode_SOD-123
- D29: renamed from D55; footprint (none) -> ScottoKeebs_Components:Diode_SOD-123
- D3: renamed from D10; footprint (none) -> ScottoKeebs_Components:Diode_SOD-123
- D30: renamed from D56; footprint (none) -> ScottoKeebs_Components:Diode_SOD-123
- D31: renamed from D57; footprint (none) -> ScottoKeebs_Components:Diode_SOD-123
- D32: renamed from D58; footprint (none) -> ScottoKeebs_Components:Diode_SOD-123
- D33: renamed from D59; footprint (none) -> ScottoKeebs_Components:Diode_SOD-123
- D34: renamed from D60; footprint (none) -> ScottoKeebs_Components:Diode_SOD-123
- D35: renamed from D61; footprint (none) -> ScottoKeebs_Components:Diode_SOD-123
- D36: renamed from D63; footprint (none) -> ScottoKeebs_Components:Diode_SOD-123
- D37: renamed from D64; footprint (none) -> ScottoKeebs_Components:Diode_SOD-123
- D38: renamed from D65; footprint (none) -> ScottoKeebs_Components:Diode_SOD-123
- D39: renamed from D66; footprint (none) -> ScottoKeebs_Components:Diode_SOD-123
- D4: renamed from D11; footprint (none) -> ScottoKeebs_Components:Diode_SOD-123
- D40: renamed from D69; footprint (none) -> ScottoKeebs_Components:Diode_SOD-123
- D41: renamed from D70; footprint (none) -> ScottoKeebs_Components:Diode_SOD-123
- D42: renamed from D72; footprint (none) -> ScottoKeebs_Components:Diode_SOD-123
- D43: renamed from D73; footprint (none) -> ScottoKeebs_Components:Diode_SOD-123
- D44: renamed from D74; footprint (none) -> ScottoKeebs_Components:Diode_SOD-123
- D45: renamed from D75; footprint (none) -> ScottoKeebs_Components:Diode_SOD-123
- D46: renamed from D76; footprint (none) -> ScottoKeebs_Components:Diode_SOD-123
- D47: renamed from D77; footprint (none) -> ScottoKeebs_Components:Diode_SOD-123
- D48: renamed from D78; footprint (none) -> ScottoKeebs_Components:Diode_SOD-123
- D49: renamed from D79; footprint (none) -> ScottoKeebs_Components:Diode_SOD-123
- D5: renamed from D12; footprint (none) -> ScottoKeebs_Components:Diode_SOD-123
- D50: renamed from D80; footprint (none) -> ScottoKeebs_Components:Diode_SOD-123
- D51: renamed from D81; footprint (none) -> ScottoKeebs_Components:Diode_SOD-123
- D52: renamed from D82; footprint (none) -> ScottoKeebs_Components:Diode_SOD-123
- D53: renamed from D83; footprint (none) -> ScottoKeebs_Components:Diode_SOD-123
- D54: renamed from D84; footprint (none) -> ScottoKeebs_Components:Diode_SOD-123
- D55: renamed from D85; footprint (none) -> ScottoKeebs_Components:Diode_SOD-123
- D56: renamed from D86; footprint (none) -> ScottoKeebs_Components:Diode_SOD-123
- D57: renamed from D87; footprint (none) -> ScottoKeebs_Components:Diode_SOD-123
- D58: renamed from D88; footprint (none) -> ScottoKeebs_Components:Diode_SOD-123
- D59: renamed from D90; footprint (none) -> ScottoKeebs_Components:Diode_SOD-123
- D6: renamed from D14; footprint (none) -> ScottoKeebs_Components:Diode_SOD-123
- D60: renamed from D91; footprint (none) -> ScottoKeebs_Components:Diode_SOD-123
- D61: renamed from D93; footprint (none) -> ScottoKeebs_Components:Diode_SOD-123
- D62: renamed from D94; footprint (none) -> ScottoKeebs_Components:Diode_SOD-123
- D63: renamed from D95; footprint (none) -> ScottoKeebs_Components:Diode_SOD-123
- D64: renamed from D96; footprint (none) -> ScottoKeebs_Components:Diode_SOD-123
- D65: renamed from D97; footprint (none) -> ScottoKeebs_Components:Diode_SOD-123
- D66: renamed from D98; footprint (none) -> ScottoKeebs_Components:Diode_SOD-123
- D67: renamed from D99; footprint (none) -> ScottoKeebs_Components:Diode_SOD-123
- D68: renamed from D100; footprint (none) -> ScottoKeebs_Components:Diode_SOD-123
- D69: renamed from D101; footprint (none) -> ScottoKeebs_Components:Diode_SOD-123
- D7: renamed from D15; footprint (none) -> ScottoKeebs_Components:Diode_SOD-123
- D70: renamed from D102; footprint (none) -> ScottoKeebs_Components:Diode_SOD-123
- D71: renamed from D103; footprint (none) -> ScottoKeebs_Components:Diode_SOD-123
- D72: renamed from D104; footprint (none) -> ScottoKeebs_Components:Diode_SOD-123
- D73: renamed from D107; footprint (none) -> ScottoKeebs_Components:Diode_SOD-123
- D74: renamed from D108; footprint (none) -> ScottoKeebs_Components:Diode_SOD-123
- D75: renamed from D112; footprint (none) -> ScottoKeebs_Components:Diode_SOD-123
- D76: renamed from D113; footprint (none) -> ScottoKeebs_Components:Diode_SOD-123
- D77: renamed from D114; footprint (none) -> ScottoKeebs_Components:Diode_SOD-123
- D78: renamed from D115; footprint (none) -> ScottoKeebs_Components:Diode_SOD-123
- D79: renamed from D116; footprint (none) -> ScottoKeebs_Components:Diode_SOD-123
- D8: renamed from D16; footprint (none) -> ScottoKeebs_Components:Diode_SOD-123
- D80: renamed from D117; footprint (none) -> ScottoKeebs_Components:Diode_SOD-123
- D81: renamed from D118; footprint (none) -> ScottoKeebs_Components:Diode_SOD-123
- D82: renamed from D119; footprint (none) -> ScottoKeebs_Components:Diode_SOD-123
- D83: renamed from D120; footprint (none) -> ScottoKeebs_Components:Diode_SOD-123
- D84: renamed from D121; footprint (none) -> ScottoKeebs_Components:Diode_SOD-123
- D85: renamed from D122; footprint (none) -> ScottoKeebs_Components:Diode_SOD-123
- D86: renamed from D123; footprint (none) -> ScottoKeebs_Components:Diode_SOD-123
- D87: renamed from D125; footprint (none) -> ScottoKeebs_Components:Diode_SOD-123
- D88: renamed from D111; footprint (none) -> ScottoKeebs_Components:Diode_SOD-123
- D89: renamed from D134; footprint (none) -> ScottoKeebs_Components:Diode_SOD-123
- D9: renamed from D17; footprint (none) -> ScottoKeebs_Components:Diode_SOD-123
- D90: renamed from D136; footprint (none) -> ScottoKeebs_Components:Diode_SOD-123
- D91: renamed from D139; footprint (none) -> ScottoKeebs_Components:Diode_SOD-123
- D92: renamed from D143; footprint (none) -> ScottoKeebs_Components:Diode_SOD-123
- D93: renamed from D144; footprint (none) -> ScottoKeebs_Components:Diode_SOD-123
- D94: renamed from D146; footprint (none) -> ScottoKeebs_Components:Diode_SOD-123
- D95: renamed from D147; footprint (none) -> ScottoKeebs_Components:Diode_SOD-123
- D96: renamed from D131; footprint (none) -> ScottoKeebs_Components:Diode_SOD-123
- D97: renamed from D132; footprint (none) -> ScottoKeebs_Components:Diode_SOD-123
- D98: renamed from D133; footprint (none) -> ScottoKeebs_Components:Diode_SOD-123
- S1: renamed from S7; footprint (none) -> ScottoKeebs_MX:MX_PCB_1.00u
- S10: renamed from S18; footprint (none) -> ScottoKeebs_MX:MX_PCB_1.00u
- S11: renamed from S19; footprint (none) -> ScottoKeebs_MX:MX_PCB_1.00u
- S12: renamed from S20; footprint (none) -> ScottoKeebs_MX:MX_PCB_1.00u
- S13: renamed from S21; footprint (none) -> ScottoKeebs_MX:MX_PCB_1.00u
- S14: renamed from S22; footprint (none) -> ScottoKeebs_MX:MX_PCB_1.00u
- S15: renamed from S23; footprint (none) -> ScottoKeebs_MX:MX_PCB_1.00u
- S16: renamed from S24; footprint (none) -> ScottoKeebs_MX:MX_PCB_1.00u
- S17: renamed from S25; footprint (none) -> ScottoKeebs_MX:MX_PCB_1.00u
- S18: renamed from S43; footprint (none) -> ScottoKeebs_MX:MX_PCB_1.00u
- S19: renamed from S44; footprint (none) -> ScottoKeebs_MX:MX_PCB_1.00u
- S2: renamed from S9; footprint (none) -> ScottoKeebs_MX:MX_PCB_1.00u
- S20: renamed from S45; footprint (none) -> ScottoKeebs_MX:MX_PCB_1.00u
- S21: renamed from S46; footprint (none) -> ScottoKeebs_MX:MX_PCB_1.00u
- S22: renamed from S48; footprint (none) -> ScottoKeebs_MX:MX_PCB_1.00u
- S23: renamed from S49; footprint (none) -> ScottoKeebs_MX:MX_PCB_1.00u
- S24: renamed from S50; footprint (none) -> ScottoKeebs_MX:MX_PCB_1.00u
- S25: renamed from S51; footprint (none) -> ScottoKeebs_MX:MX_PCB_1.00u
- S26: renamed from S52; footprint (none) -> ScottoKeebs_MX:MX_PCB_1.00u
- S27: renamed from S53; footprint (none) -> ScottoKeebs_MX:MX_PCB_1.00u
- S28: renamed from S54; footprint (none) -> ScottoKeebs_MX:MX_PCB_1.00u
- S29: renamed from S55; footprint (none) -> ScottoKeebs_MX:MX_PCB_1.00u
- S3: renamed from S10; footprint (none) -> ScottoKeebs_MX:MX_PCB_1.00u
- S30: renamed from S56; footprint (none) -> ScottoKeebs_MX:MX_PCB_1.00u
- S31: renamed from S57; footprint (none) -> ScottoKeebs_MX:MX_PCB_1.00u
- S32: renamed from S58; footprint (none) -> ScottoKeebs_MX:MX_PCB_1.00u
- S33: renamed from S59; footprint (none) -> ScottoKeebs_MX:MX_PCB_1.00u
- S34: renamed from S60; footprint (none) -> ScottoKeebs_MX:MX_PCB_1.00u
- S35: renamed from S61; footprint (none) -> ScottoKeebs_MX:MX_PCB_1.00u
- S36: renamed from S63; footprint (none) -> ScottoKeebs_MX:MX_PCB_1.00u
- S37: renamed from S64; footprint (none) -> ScottoKeebs_MX:MX_PCB_1.00u
- S38: renamed from S65; footprint (none) -> ScottoKeebs_MX:MX_PCB_1.00u
- S39: renamed from S66; footprint (none) -> ScottoKeebs_MX:MX_PCB_1.00u
- S4: renamed from S11; footprint (none) -> ScottoKeebs_MX:MX_PCB_1.00u
- S40: renamed from S69; footprint (none) -> ScottoKeebs_MX:MX_PCB_1.00u
- S41: renamed from S70; footprint (none) -> ScottoKeebs_MX:MX_PCB_1.00u
- S42: renamed from S72; footprint (none) -> ScottoKeebs_MX:MX_PCB_1.00u
- S43: renamed from S73; footprint (none) -> ScottoKeebs_MX:MX_PCB_1.00u
- S44: renamed from S74; footprint (none) -> ScottoKeebs_MX:MX_PCB_1.00u
- S45: renamed from S75; footprint (none) -> ScottoKeebs_MX:MX_PCB_1.00u
- S46: renamed from S76; footprint (none) -> ScottoKeebs_MX:MX_PCB_1.00u
- S47: renamed from S77; footprint (none) -> ScottoKeebs_MX:MX_PCB_1.00u
- S48: renamed from S78; footprint (none) -> ScottoKeebs_MX:MX_PCB_1.00u
- S49: renamed from S79; footprint (none) -> ScottoKeebs_MX:MX_PCB_1.00u
- S5: renamed from S12; footprint (none) -> ScottoKeebs_MX:MX_PCB_1.00u
- S50: renamed from S80; footprint (none) -> ScottoKeebs_MX:MX_PCB_1.00u
- S51: renamed from S81; footprint (none) -> ScottoKeebs_MX:MX_PCB_1.00u
- S52: renamed from S82; footprint (none) -> ScottoKeebs_MX:MX_PCB_1.00u
- S53: renamed from S83; footprint (none) -> ScottoKeebs_MX:MX_PCB_1.00u
- S54: renamed from S84; footprint (none) -> ScottoKeebs_MX:MX_PCB_1.00u
- S55: renamed from S85; footprint (none) -> ScottoKeebs_MX:MX_PCB_1.00u
- S56: renamed from S86; footprint (none) -> ScottoKeebs_MX:MX_PCB_1.00u
- S57: renamed from S87; footprint (none) -> ScottoKeebs_MX:MX_PCB_1.00u
- S58: renamed from S88; footprint (none) -> ScottoKeebs_MX:MX_PCB_1.00u
- S59: renamed from S90; footprint (none) -> ScottoKeebs_MX:MX_PCB_1.00u
- S6: renamed from S14; footprint (none) -> ScottoKeebs_MX:MX_PCB_1.00u
- S60: renamed from S91; footprint (none) -> ScottoKeebs_MX:MX_PCB_1.00u
- S61: renamed from S93; footprint (none) -> ScottoKeebs_MX:MX_PCB_1.00u
- S62: renamed from S94; footprint (none) -> ScottoKeebs_MX:MX_PCB_1.00u
- S63: renamed from S95; footprint (none) -> ScottoKeebs_MX:MX_PCB_1.00u
- S64: renamed from S96; footprint (none) -> ScottoKeebs_MX:MX_PCB_1.00u
- S65: renamed from S97; footprint (none) -> ScottoKeebs_MX:MX_PCB_1.00u
- S66: renamed from S98; footprint (none) -> ScottoKeebs_MX:MX_PCB_1.00u
- S67: renamed from S99; footprint (none) -> ScottoKeebs_MX:MX_PCB_1.00u
- S68: renamed from S100; footprint (none) -> ScottoKeebs_MX:MX_PCB_1.00u
- S69: renamed from S101; footprint (none) -> ScottoKeebs_MX:MX_PCB_1.00u
- S7: renamed from S15; footprint (none) -> ScottoKeebs_MX:MX_PCB_1.00u
- S70: renamed from S102; footprint (none) -> ScottoKeebs_MX:MX_PCB_1.00u
- S71: renamed from S103; footprint (none) -> ScottoKeebs_MX:MX_PCB_1.00u
- S72: renamed from S104; footprint (none) -> ScottoKeebs_MX:MX_PCB_1.00u
- S73: renamed from S107; footprint (none) -> ScottoKeebs_MX:MX_PCB_1.00u
- S74: renamed from S108; footprint (none) -> ScottoKeebs_MX:MX_PCB_1.00u
- S75: renamed from S112; footprint (none) -> ScottoKeebs_MX:MX_PCB_1.00u
- S76: renamed from S113; footprint (none) -> ScottoKeebs_MX:MX_PCB_1.00u
- S77: renamed from S114; footprint (none) -> ScottoKeebs_MX:MX_PCB_1.00u
- S78: renamed from S115; footprint (none) -> ScottoKeebs_MX:MX_PCB_1.00u
- S79: renamed from S116; footprint (none) -> ScottoKeebs_MX:MX_PCB_1.00u
- S8: renamed from S16; footprint (none) -> ScottoKeebs_MX:MX_PCB_1.00u
- S80: renamed from S117; footprint (none) -> ScottoKeebs_MX:MX_PCB_1.00u
- S81: renamed from S118; footprint (none) -> ScottoKeebs_MX:MX_PCB_1.00u
- S82: renamed from S119; footprint (none) -> ScottoKeebs_MX:MX_PCB_1.00u
- S83: renamed from S120; footprint (none) -> ScottoKeebs_MX:MX_PCB_1.00u
- S84: renamed from S121; footprint (none) -> ScottoKeebs_MX:MX_PCB_1.00u
- S85: renamed from S122; footprint (none) -> ScottoKeebs_MX:MX_PCB_1.00u
- S86: renamed from S123; footprint (none) -> ScottoKeebs_MX:MX_PCB_1.00u
- S87: renamed from S125; footprint (none) -> ScottoKeebs_MX:MX_PCB_1.00u
- S88: renamed from S111; footprint (none) -> ScottoKeebs_MX:MX_PCB_1.00u
- S89: renamed from S134; footprint (none) -> ScottoKeebs_MX:MX_PCB_1.00u
- S9: renamed from S17; footprint (none) -> ScottoKeebs_MX:MX_PCB_1.00u
- S90: renamed from S136; footprint (none) -> ScottoKeebs_MX:MX_PCB_1.00u
- S91: renamed from S139; footprint (none) -> ScottoKeebs_MX:MX_PCB_1.00u
- S92: renamed from S143; footprint (none) -> ScottoKeebs_MX:MX_PCB_1.00u
- S93: renamed from S144; footprint (none) -> ScottoKeebs_MX:MX_PCB_1.00u
- S94: renamed from S146; footprint (none) -> ScottoKeebs_MX:MX_PCB_1.00u
- S95: renamed from S147; footprint (none) -> ScottoKeebs_MX:MX_PCB_1.00u
- S96: renamed from S131; footprint (none) -> ScottoKeebs_MX:MX_PCB_1.00u
- S97: renamed from S132; footprint (none) -> ScottoKeebs_MX:MX_PCB_1.00u
- S98: renamed from S133; footprint (none) -> ScottoKeebs_MX:MX_PCB_1.00u
- U1: footprint 44PW_ATM -> Microchip Tech ATMEGA32U4-MU:44PW_ATM
- renumbered C1 to C3, C2 to C4, SW1 to R_BUTT1
Connections:
- net COL_1: now also U1.18 (PD0)
- net COL_2: now also U1.19 (PD1)
- net COL_3: now also U1.20 (PD2)
- net COL_4: now also U1.21 (PD3)
- net COL_5: now also U1.25 (PD4)
- net COL_6: now also U1.22 (PD5)
- net COL_7: now also U1.26 (PD6)
- net COL_8: now also U1.27 (PD7)
- net GND: now also U1.15 (GND), U1.23 (GND), U1.35 (GND), U1.43 (GND), C1.1, C2.1
- net VCC: now reaches U1.14 (VCC)
- net VCC: now also U1.34 (VCC), FB1.2, FB2.2
- net AVCC1: now reaches U1.24 (AVCC)
- net AVCC1: now also C2.2, FB2.1
- net AVCC2: now reaches U1.44 (AVCC)
- net AVCC2: now also C1.2, FB1.1
Other:
- moved on the sheet: D1, D10, D11, D12, D13, D14, D15, D16, D17, D18, D19, D2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
